Commit message: no more gazebo needed

File: robot_models/franka_gazebo/urdf/panda_arm.gazebo_ros2_control.xacro (robot description, xacro)
@@ -3,49 +3,13 @@
   <xacro:include filename="$(find franka_gazebo)/urdf/materials.xacro" />
   <xacro:macro name="panda_arm_gazebo_ros2_control" params="ns hand:='false'">
-    <gazebo>
-      <plugin filename="libgazebo_ros2_control.so" name="gazebo_ros2_control">
-        <parameters>$(find franka_gazebo)/config/franka_controllers.yaml</parameters>
-      </plugin>
-    </gazebo>
-    <!-- Links -->
-    <xacro:macro name="configure_link" params="link_name">
-    <gazebo reference="${link_name}">
-      <material>Gazebo/White</material>
-      <selfCollide>False</selfCollide>
-    </gazebo>
-    </xacro:macro>
-    <xacro:configure_link link_name="${ns}_link0"/>
-    <xacro:configure_link link_name="${ns}_link1"/>
-    <xacro:configure_link link_name="${ns}_link2"/>
-    <xacro:configure_link link_name="${ns}_link3"/>
-    <xacro:configure_link link_name="${ns}_link4"/>
-    <xacro:configure_link link_name="${ns}_link5"/>
-    <xacro:configure_link link_name="${ns}_link6"/>
-    <xacro:configure_link link_name="${ns}_link7"/>
-    <!--xacro:configure_link link_name="${ns}_link8"/-->
-    <xacro:macro name="configure_joint_ref" params="joint_name">
-    <gazebo reference="${joint_name}">
-      <implicitSpringDamper>True</implicitSpringDamper>
-    </gazebo>
-    </xacro:macro>
-    <xacro:configure_joint_ref joint_name="${ns}_joint1"/>
-    <xacro:configure_joint_ref joint_name="${ns}_joint2"/>
-    <xacro:configure_joint_ref joint_name="${ns}_joint3"/>
-    <xacro:configure_joint_ref joint_name="${ns}_joint4"/>
-    <xacro:configure_joint_ref joint_name="${ns}_joint5"/>
-    <xacro:configure_joint_ref joint_name="${ns}_joint6"/>
-    <xacro:configure_joint_ref joint_name="${ns}_joint7"/>
-    <xacro:if value="${hand == 'true'}">
-    <xacro:configure_link link_name="${ns}_link6"/>
-      <xacro:configure_link link_name="${ns}_hand"/>
-      <xacro:configure_link link_name="${ns}_hand_tcp"/>
-      <xacro:configure_link link_name="${ns}_leftfinger"/>
-      <xacro:configure_link link_name="${ns}_rightfinger"/>
-      <xacro:configure_joint_ref joint_name="${ns}_finger_joint1"/>
-      <xacro:configure_joint_ref joint_name="${ns}_finger_joint2"/>
-    </xacro:if>
     <ros2_control name="FrankaHardwareInterface" type="system">
       <hardware>
-        <plugin>gazebo_ros2_control/GazeboSystem</plugin>
+        <plugin>mock_components/GenericSystem</plugin>
+        <param name="calculate_dynamics">true</param>
+        <param name="custom_interface_with_following_offset"></param>
+        <param name="disable_commands">false</param>
+        <param name="mock_gpio_commands">false</param>
+        <param name="mock_sensor_commands">false</param>
+        <param name="position_state_following_offset">0.0</param>
       </hardware>
       <xacro:macro name="configure_joint" params="joint_name initial_position min_vel max_vel">

File: robot_models/rrbot/urdf/rrbot.urdf.xacro (robot description, xacro)
@@ -16,30 +16,14 @@
     <origin xyz="0 0 0" rpy="0 0 0" />
   </xacro:rrbot>
-  <!-- gazebo ros_control stuff-->
-  <gazebo>
-    <plugin filename="libgazebo_ros2_control.so" name="gazebo_ros2_control">
-      <parameters>$(find rrbot)/config/rrbot_controllers.yaml</parameters>
-    </plugin>
-  </gazebo>
-  <!-- Link1 -->
-  <gazebo reference="$(arg prefix)base_link">
-    <material>Gazebo/Orange</material>
-  </gazebo>
-  <!-- Link2 -->
-  <gazebo reference="$(arg prefix)link1">
-    <mu1>0.2</mu1>
-    <mu2>0.2</mu2>
-    <material>Gazebo/Yellow</material>
-  </gazebo>
-  <!-- Link3 -->
-  <gazebo reference="$(arg prefix)link2">
-    <mu1>0.2</mu1>
-    <mu2>0.2</mu2>
-    <material>Gazebo/Orange</material>
-  </gazebo>
   <!-- ros_control plugin -->
   <ros2_control name="RRBot" type="system">
     <hardware>
-      <plugin>gazebo_ros2_control/GazeboSystem</plugin>
+      <plugin>mock_components/GenericSystem</plugin>
+      <param name="calculate_dynamics">true</param>
+      <param name="custom_interface_with_following_offset"></param>
+      <param name="disable_commands">false</param>
+      <param name="mock_gpio_commands">false</param>
+      <param name="mock_sensor_commands">false</param>
+      <param name="position_state_following_offset">0.0</param>
     </hardware>
     <joint name="joint1">
